File: Eagle Files/rs485board/rs485board.brd (EAGLE design)
At the start: 63.2 x 63.5 mm, 59 parts, among them IC1 XC6206P332MR, IC2 MP2359, J1 AVR_SPI_PROG_3X2PTH, J2 RA 6Pin SMD, Q1 CJ3404, Q2 CJ3404, Q3 CJ3404, U1 ATMEGA328P_TQFP, U2 LIS3DH, U3 MAX3485CSA, X1 RJ45-8L-B, X2 RJ45-8L-B, Y1 16MHz

Commit message: add more traces
Parts:
- added C14, C15, C16, C17, C18, C19, C20, C21, C22, C23, C24, C25, C26: (no value), resistor:C0805K
- added J6: (no value), SparkFun-Connectors:1X01
- added PAD1, PAD2: (no value), wirepad:1,6/0,8
- added R11, R12, R13: (no value), resistor:R0805
- moved R7 71.3 mm to (3.05, 28.7), turned to 180 degrees
- moved D4 70.9 mm to (2.03, 23.9), turned to 90 degrees
- moved R6 70.0 mm to (3.05, 31.2), turned to 180 degrees
- moved D2 68.3 mm to (4.06, 23.9), turned to 90 degrees
- moved D3 66.5 mm to (6.10, 23.9), turned to 90 degrees
- moved D1 64.9 mm to (8.13, 23.9), turned to 90 degrees
- moved D5 64.5 mm to (11.7, 32.8), turned to 90 degrees
- moved D6 61.3 mm to (9.91, 32.8), turned to 90 degrees
- moved Q3 11.2 mm to (41.9, 3.05)
- moved C6 9.88 mm to (2.03, 37.6), turned to 270 degrees
- moved R5 9.68 mm to (3.05, 33.8), turned to 180 degrees
- moved J3 9.25 mm to (33.0, 8.89)
- moved C12 8.64 mm to (40.6, 60.7)
- moved J4 8.03 mm to (38.1, 8.89)
- moved C11 7.94 mm to (35.6, 60.7), turned to 180 degrees
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Connections:
- new net +5V6: C14.1, D7.1
- new net A0: U1.23
- new net A1: U1.24
- new net A2: U1.25
- new net A3: U1.26
- new net A4: U1.27
- new net A5: U1.28
- new net A6: U1.19
- new net A7: U1.22
- new net D7: PAD1.1, U1.11
- new net D8: PAD2.1, U1.12
- new net DIR: U1.2, U3.2, U3.3
- new net N$20: R11.2, U3.7, X1.1, X2.1
- new net N$22: R11.1, U3.6, X1.2, X2.2
- new net N$30: R12.2, U3.1
- new net N$31: R13.2, U3.4
- net +24V: now also X1.4, X1.5, X2.4, X2.5
- net +3V3: no longer C2.1, C3.1, C4.1, U1.18, U1.4, U1.6
- net +5V: now also C15.1, C16.1, C17.1, C18.1, C19.1, C2.1, C20.1, C21.1, C22.1, C23.1, C24.1, C25.1, C26.1, C3.1, C4.1, D10.1, D11.1, D12.1, D13.1, D14.1, D15.1, D16.1, D17.1, D18.1, D8.1, D9.1, J6.1, U1.18, U1.4, U1.6, U3.8
- net GND: now also C14.2, C15.2, C16.2, C17.2, C18.2, C19.2, C20.2, C21.2, C22.2, C23.2, C24.2, C25.2, C26.2, D10.3, D11.3, D12.3, D13.3, D14.3, D15.3, D16.3, D17.3, D18.3, D7.3, D8.3, D9.3, U3.5, X1.3, X1.6, X1.7, X1.8, X2.3, X2.6, X2.7, X2.8
- net RX: now also R12.1
- net TX: now also R13.1
Routing:
- net GND: track 0.00 -> 434.4 mm, vias 0 -> 29
- net +5V: track 0.00 -> 257.8 mm, vias 0 -> 4
- net TX: track 0.00 -> 75.9 mm, vias 0 -> 2
- net RX: track 0.00 -> 68.0 mm, vias 0 -> 2
- net DIR: track 0.00 -> 64.4 mm, vias 0 -> 2
- net MOSI: track 0.00 -> 58.4 mm, vias 0 -> 3
- net D5: track 0.00 -> 48.5 mm, vias 0 -> 2
- net SCK: track 0.00 -> 45.6 mm, vias 0 -> 3
- net RESET_EXT: track 0.00 -> 44.1 mm, vias 0 -> 2
- net D6: track 0.00 -> 43.1 mm, vias 0 -> 2
- net MISO: track 0.00 -> 41.7 mm, vias 0 -> 2
- net D9: track 0.00 -> 30.5 mm
- net RESET: track 0.00 -> 29.8 mm
- net +3V3: track 0.00 -> 25.4 mm
- net SS: track 0.00 -> 22.6 mm, vias 0 -> 2
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Other:
- board size 63.2 x 63.5 mm -> 63.5 x 63.5 mm

Commit message: add more traces
Parts:
- added PAD3, PAD4, PAD5: (no value), wirepad:1,6/0,8
- moved C6 34.8 mm to (36.3, 31.8), turned to 90 degrees
- moved C7 27.5 mm to (31.8, 36.1), turned to 180 degrees
- moved U2 24.3 mm to (31.8, 31.8), turned to 270 degrees
- moved C8 13.0 mm to (3.56, 34.3), turned to 270 degrees
- moved C26 10.7 mm to (52.3, 37.3), turned to 270 degrees
- moved C9 9.43 mm to (10.7, 34.3), turned to 270 degrees
- moved C12 9.40 mm to (37.6, 51.8), turned to 180 degrees
- moved D5 8.95 mm to (12.7, 23.9)
- moved D6 8.90 mm to (10.4, 23.9)
- moved IC1 8.84 mm to (7.11, 34.3), turned to 90 degrees
- moved R5 6.83 mm to (8.13, 29.2), turned to 90 degrees
- moved X2 4.37 mm to (52.1, 53.6), flipped to the bottom, turned to 160 degrees
- moved X1 3.94 mm to (11.2, 53.3), flipped to the bottom, turned to 200 degrees
- moved R6 2.87 mm to (5.08, 29.2), turned to 90 degrees
- moved R7 1.14 mm to (2.03, 29.2), turned to 90 degrees
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Connections:
- net N$20 renamed RS485B
- net N$22 renamed RS485A
- removed net +5V6: C14.1, D7.1
- net +5V: now also C14.1, D7.1
- net A3: now also D7.4
- net A4: now also PAD3.1
- net A5: now also PAD4.1
- net GND: now also PAD5.1
Routing:
- net GND: track 434.4 -> 651.6 mm
- net +5V: track 257.8 -> 380.6 mm, vias 4 -> 10
- net RS485B: track 3.68 -> 66.4 mm, vias 0 -> 1
- net RS485A: track 3.68 -> 65.1 mm, vias 0 -> 1
- net +24V: track 8.85 -> 69.8 mm, vias 0 -> 1
- net +3V3: track 25.4 -> 60.3 mm, vias 0 -> 2
- net A3: track 0.00 -> 20.9 mm, vias 0 -> 2
- net INT2: track 2.77 -> 22.6 mm, vias 0 -> 2
- net SCK_3.3V: track 22.0 -> 41.0 mm
- net INT1: track 4.72 -> 22.3 mm, vias 0 -> 2
- net MISO_3.3V: track 11.7 -> 27.6 mm, vias 0 -> 2
- net MOSI_3.3V: track 16.8 -> 32.6 mm
- net SS_3.3V: track 15.5 -> 26.6 mm
- net D2: track 17.2 -> 7.92 mm
- net D3: track 16.1 -> 7.39 mm
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Other:
- outline, holes or cut-outs redrawn

Commit message: adjust wires
Parts:
- removed X2: RJ45-8L-B, con-tycoelectronics:RJ45-NO-SHIELD
- added X3: RJ45-8P8C-8L-B, myownParts:RJ45-SHIELD-DS1128-S80BP
- X1: value RJ45-8L-B -> RJ45-8P8C-8L-B; device con-tycoelectronics:RJ45-NO-SHIELD -> myownParts:RJ45-SHIELD-DS1128-S80BP
- moved X1 40.9 mm to (52.1, 53.3), turned to 160 degrees
Connections:
- net +24V: now also X3.4, X3.5; no longer X2.4, X2.5
- net GND: now also X3.3, X3.6, X3.7, X3.8; no longer X2.3, X2.6, X2.7, X2.8
- net RS485A: now also X3.2; no longer X2.2
- net RS485B: now also X3.1; no longer X2.1
Routing:
- net GND: track 651.6 -> 623.1 mm, vias 29 -> 31
- net +5V: track 380.6 -> 364.3 mm, vias 10 -> 11
Other:
- outline, holes or cut-outs redrawn
