File: Eagle Files/rs485board/rs485board.sch (EAGLE design)
At the start: 59 parts, among them IC1 XC6206P332MR, IC2 MP2359, J1 AVR_SPI_PROG_3X2PTH, J2 RA 6Pin SMD, Q1 CJ3404, Q2 CJ3404, Q3 CJ3404, U1 ATMEGA328P_TQFP, U2 LIS3DH, U3 MAX3485CSA, X1 RJ45-8L-B, X2 RJ45-8L-B, Y1 16MHz

Commit message: add more traces
Parts:
- added C14, C15, C16, C17, C18, C19, C20, C21, C22, C23, C24, C25, C26: (no value), resistor:C-EUC0805K
- added J6: (no value), SparkFun-Connectors:CONN_01
- added PAD1, PAD2: (no value), wirepad:1,6/0,8
- added R11, R12, R13: (no value), resistor:R-US_R0805
Connections:
- new net +5V6: C14.1, D7.VDD
- new net A0: U1.PC0(ADC0)
- new net A1: U1.PC1(ADC1)
- new net A2: U1.PC2(ADC2)
- new net A3: U1.PC3(ADC3)
- new net A4: U1.PC4(ADC4/SDA)
- new net A5: U1.PC5(ADC5/SCL)
- new net A6: U1.ADC6
- new net A7: U1.ADC7
- new net D7: PAD1.P, U1.PD7(AIN1)
- new net D8: PAD2.P, U1.PB0(ICP)
- new net DIR: U1.PD4(XCK/T0), U3./RE, U3.DE
- new net N$20: R11.2, U3.B, X1.1, X2.1
- new net N$22: R11.1, U3.A, X1.2, X2.2
- new net N$30: R12.2, U3.RO
- new net N$31: R13.2, U3.DI
- net +24V: now also X1.4, X1.5, X2.4, X2.5
- net +3V3: no longer C2.1, C3.1, C4.1, U1.AVCC, U1.VCC@4, U1.VCC@6
- net +5V: now also C15.1, C16.1, C17.1, C18.1, C19.1, C2.1, C20.1, C21.1, C22.1, C23.1, C24.1, C25.1, C26.1, C3.1, C4.1, D10.VDD, D11.VDD, D12.VDD, D13.VDD, D14.VDD, D15.VDD, D16.VDD, D17.VDD, D18.VDD, D8.VDD, D9.VDD, J6.1, U1.AVCC, U1.VCC@4, U1.VCC@6, U3.VCC
- net GND: now also C14.2, C15.2, C16.2, C17.2, C18.2, C19.2, C20.2, C21.2, C22.2, C23.2, C24.2, C25.2, C26.2, D10.VSS, D11.VSS, D12.VSS, D13.VSS, D14.VSS, D15.VSS, D16.VSS, D17.VSS, D18.VSS, D7.VSS, D8.VSS, D9.VSS, U3.GND, X1.3, X1.6, X1.7, X1.8, X2.3, X2.6, X2.7, X2.8
- net RX: now also R12.1
- net TX: now also R13.1
Other:
- moved on the sheet: U3, X1, X2

Commit message: add more traces
Parts:
- added PAD3, PAD4, PAD5: (no value), wirepad:1,6/0,8
Connections:
- net N$20 renamed RS485B
- net N$22 renamed RS485A
- removed net +5V6: C14.1, D7.VDD
- net +5V: now also C14.1, D7.VDD
- net A3: now also D7.DI
- net A4: now also PAD3.P
- net A5: now also PAD4.P
- net GND: now also PAD5.P
Changed lines of the file:
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@@
 <part name="GND15" library="SparkFun-PowerSymbols" deviceset="GND" device=""/>
 <part name="P+9" library="supply1" library_urn="urn:adsk.eagle:library:371" deviceset="+5V" device=""/>
+<part name="PAD3" library="wirepad" library_urn="urn:adsk.eagle:library:412" deviceset="1,6/0,8" device="" package3d_urn="urn:adsk.eagle:package:30830/1"/>
+<part name="PAD4" library="wirepad" library_urn="urn:adsk.eagle:library:412" deviceset="1,6/0,8" device="" package3d_urn="urn:adsk.eagle:package:30830/1"/>
+<part name="PAD5" library="wirepad" library_urn="urn:adsk.eagle:library:412" deviceset="1,6/0,8" device="" package3d_urn="urn:adsk.eagle:package:30830/1"/>
+<part name="GND17" library="SparkFun-PowerSymbols" deviceset="GND" device=""/>
 </parts>
 <sheets>
@@
 <instance part="D1" gate="G$1" x="106.68" y="27.94" rot="R180"/>
 <instance part="R5" gate="G$1" x="147.32" y="35.56" rot="R90"/>
-<instance part="+3V2" gate="G$1" x="147.32" y="45.72"/>
+<instance part="+3V2" gate="G$1" x="147.32" y="43.18"/>
 <instance part="D2" gate="G$1" x="109.22" y="25.4" rot="R180"/>
 <instance part="D3" gate="G$1" x="111.76" y="22.86" rot="R180"/>
 <instance part="D4" gate="G$1" x="114.3" y="20.32" rot="R180"/>
 <instance part="R6" gate="G$1" x="142.24" y="35.56" rot="R90"/>
-<instance part="+3V3" gate="G$1" x="142.24" y="45.72"/>
+<instance part="+3V3" gate="G$1" x="142.24" y="43.18"/>
 <instance part="R7" gate="G$1" x="137.16" y="35.56" rot="R90"/>
-<instance part="+3V6" gate="G$1" x="137.16" y="45.72"/>
+<instance part="+3V6" gate="G$1" x="137.16" y="43.18"/>
 <instance part="D5" gate="G$1" x="81.28" y="50.8" rot="R180"/>
 <instance part="D6" gate="G$1" x="91.44" y="48.26" rot="R180"/>
@@
 <instance part="GND15" gate="1" x="-111.76" y="-33.02"/>
 <instance part="P+9" gate="1" x="-109.22" y="81.28"/>
+<instance part="PAD3" gate="P" x="71.12" y="68.58" smashed="yes" rot="R180">
+<attribute name="NAME" x="79.883" y="69.2658" size="1.778" layer="95" rot="R180"/>
+<attribute name="VALUE" x="72.263" y="71.882" size="1.778" layer="96" rot="R180"/>
+</instance>
+<instance part="PAD4" gate="P" x="71.12" y="66.04" smashed="yes" rot="R180">
+<attribute name="NAME" x="79.883" y="66.7258" size="1.778" layer="95" rot="R180"/>
+<attribute name="VALUE" x="72.263" y="69.342" size="1.778" layer="96" rot="R180"/>
+</instance>
+<instance part="PAD5" gate="P" x="73.66" y="83.82" smashed="yes" rot="R180">
+<attribute name="NAME" x="82.423" y="84.5058" size="1.778" layer="95" rot="R180"/>
+<attribute name="VALUE" x="74.803" y="87.122" size="1.778" layer="96" rot="R180"/>
+</instance>
+<instance part="GND17" gate="1" x="71.12" y="81.28"/>
 </instances>
 <busses>
@@
 <pinref part="GND29" gate="1" pin="GND"/>
 <junction x="-40.64" y="-60.96"/>
+<junction x="-38.1" y="-60.96"/>
 </segment>
 <segment>
@@
 <junction x="-111.76" y="-30.48"/>
 </segment>
+<segment>
+<pinref part="PAD5" gate="P" pin="P"/>
+<pinref part="GND17" gate="1" pin="GND"/>
+</segment>
 </net>
 <net name="RESET_EXT" class="0">
@@
 <pinref part="+3V2" gate="G$1" pin="+3V3"/>
 <pinref part="R5" gate="G$1" pin="2"/>
-<wire x1="147.32" y1="43.18" x2="147.32" y2="40.64" width="0.1524" layer="91"/>
 </segment>
 <segment>
 <pinref part="+3V3" gate="G$1" pin="+3V3"/>
 <pinref part="R6" gate="G$1" pin="2"/>
-<wire x1="142.24" y1="43.18" x2="142.24" y2="40.64" width="0.1524" layer="91"/>
 </segment>
 <segment>
 <pinref part="+3V6" gate="G$1" pin="+3V3"/>
 <pinref part="R7" gate="G$1" pin="2"/>
-<wire x1="137.16" y1="43.18" x2="137.16" y2="40.64" width="0.1524" layer="91"/>
 </segment>
 </net>
@@
 <junction x="-106.68" y="-22.86"/>
 <pinref part="P+9" gate="1" pin="+5V"/>
+<pinref part="D7" gate="G$1" pin="VDD"/>
+<pinref part="C14" gate="G$1" pin="1"/>
+<wire x1="-109.22" y1="78.74" x2="-106.68" y2="78.74" width="0.1524" layer="91"/>
+<junction x="-109.22" y="78.74"/>
+<junction x="-106.68" y="78.74"/>
 </segment>
 </net>
@@
 <wire x1="63.5" y1="66.04" x2="68.58" y2="66.04" width="0.1524" layer="91"/>
 <label x="66.04" y="66.04" size="1.778" layer="95"/>
+<pinref part="PAD4" gate="P" pin="P"/>
 </segment>
 </net>
@@
 <wire x1="63.5" y1="68.58" x2="68.58" y2="68.58" width="0.1524" layer="91"/>
 <label x="66.04" y="68.58" size="1.778" layer="95"/>
+<pinref part="PAD3" gate="P" pin="P"/>
 </segment>
 </net>
@@
 <wire x1="63.5" y1="71.12" x2="68.58" y2="71.12" width="0.1524" layer="91"/>
 <label x="66.04" y="71.12" size="1.778" layer="95"/>
+</segment>
+<segment>
+<pinref part="D7" gate="G$1" pin="DI"/>
+<wire x1="-78.74" y1="78.74" x2="-78.74" y2="88.9" width="0.1524" layer="91"/>
+<wire x1="-78.74" y1="88.9" x2="-73.66" y2="88.9" width="0.1524" layer="91"/>
+<label x="-78.74" y="88.9" size="1.778" layer="95"/>
 </segment>
 </net>
@@
 </segment>
 </net>
-<net name="N$20" class="0">
+<net name="RS485B" class="0">
 <segment>
 <pinref part="U3" gate="G$1" pin="B"/>
@@
 </segment>
 </net>
-<net name="N$22" class="0">
+<net name="RS485A" class="0">
 <segment>
 <pinref part="U3" gate="G$1" pin="A"/>
@@
 </segment>
 </net>
-<net name="+5V6" class="0">
-<segment>
-<wire x1="-106.68" y1="78.74" x2="-109.22" y2="78.74" width="0.1524" layer="91"/>
-<pinref part="D7" gate="G$1" pin="VDD"/>
-<pinref part="C14" gate="G$1" pin="1"/>
-<junction x="-106.68" y="78.74"/>
-</segment>
-</net>

Commit message: adjust wires
Parts:
- removed X2: RJ45-8L-B, con-tycoelectronics:RJ45-8L-B
- added X3: RJ45-8P8C-8L-B, myownParts:RJ45-8P8C-8L-B
- X1: value RJ45-8L-B -> RJ45-8P8C-8L-B; device con-tycoelectronics:RJ45-8L-B -> myownParts:RJ45-8P8C-8L-B
Connections:
- net +24V: now also X3.4, X3.5; no longer X2.4, X2.5
- net GND: now also X3.3, X3.6, X3.7, X3.8; no longer X2.3, X2.6, X2.7, X2.8
- net RS485A: now also X3.2; no longer X2.2
- net RS485B: now also X3.1; no longer X2.1
Other:
- moved on the sheet: X1
Changed lines of the file:
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@@
 <part name="D5" library="adafruit" library_urn="urn:adsk.eagle:library:420" deviceset="DIODE" device="SOD-123"/>
 <part name="D6" library="adafruit" library_urn="urn:adsk.eagle:library:420" deviceset="DIODE" device="SOD-123"/>
-<part name="X1" library="con-tycoelectronics" library_urn="urn:adsk.eagle:library:193" deviceset="RJ45" device="" package3d_urn="urn:adsk.eagle:package:10660/1" technology="-8L-B"/>
-<part name="X2" library="con-tycoelectronics" library_urn="urn:adsk.eagle:library:193" deviceset="RJ45" device="" package3d_urn="urn:adsk.eagle:package:10660/1" technology="-8L-B"/>
 <part name="U3" library="SparkFun-IC-Comms" deviceset="RS485" device="SOIC" value=" MAX3485CSA"/>
 <part name="D7" library="SparkFun-LED" library_urn="urn:adsk.eagle:library:529" deviceset="WS2812B" device="" package3d_urn="urn:adsk.eagle:package:39369/1" value="WS2812B"/>
@@
 <part name="PAD5" library="wirepad" library_urn="urn:adsk.eagle:library:412" deviceset="1,6/0,8" device="" package3d_urn="urn:adsk.eagle:package:30830/1"/>
 <part name="GND17" library="SparkFun-PowerSymbols" deviceset="GND" device=""/>
+<part name="X3" library="myownParts" deviceset="RJ45-8P8C" device="" technology="-8L-B"/>
+<part name="X1" library="myownParts" deviceset="RJ45-8P8C" device="" technology="-8L-B"/>
 </parts>
 <sheets>
@@
 <instance part="D5" gate="G$1" x="81.28" y="50.8" rot="R180"/>
 <instance part="D6" gate="G$1" x="91.44" y="48.26" rot="R180"/>
-<instance part="X1" gate="G$1" x="-35.56" y="-55.88"/>
-<instance part="X2" gate="G$1" x="-20.32" y="-55.88"/>
 <instance part="U3" gate="G$1" x="-71.12" y="-55.88"/>
 <instance part="D7" gate="G$1" x="-91.44" y="73.66"/>
@@
 </instance>
 <instance part="GND17" gate="1" x="71.12" y="81.28"/>
+<instance part="X3" gate="G$1" x="-35.56" y="-55.88"/>
+<instance part="X1" gate="G$1" x="-20.32" y="-55.88"/>
 </instances>
 <busses>
@@
 </segment>
 <segment>
-<pinref part="X1" gate="G$1" pin="7"/>
-<pinref part="X1" gate="G$1" pin="8"/>
 <wire x1="-38.1" y1="-63.5" x2="-38.1" y2="-66.04" width="0.1524" layer="91"/>
-<pinref part="X2" gate="G$1" pin="7"/>
-<pinref part="X2" gate="G$1" pin="8"/>
 <wire x1="-22.86" y1="-63.5" x2="-22.86" y2="-66.04" width="0.1524" layer="91"/>
 <wire x1="-38.1" y1="-66.04" x2="-22.86" y2="-66.04" width="0.1524" layer="91"/>
@@
 <junction x="-22.86" y="-66.04"/>
 <pinref part="GND28" gate="1" pin="GND"/>
-</segment>
-<segment>
-<pinref part="X1" gate="G$1" pin="3"/>
+<pinref part="X3" gate="G$1" pin="7"/>
+<pinref part="X3" gate="G$1" pin="8"/>
+<pinref part="X1" gate="G$1" pin="7"/>
+<pinref part="X1" gate="G$1" pin="8"/>
+</segment>
+<segment>
 <wire x1="-38.1" y1="-53.34" x2="-40.64" y2="-53.34" width="0.1524" layer="91"/>
 <wire x1="-40.64" y1="-53.34" x2="-40.64" y2="-60.96" width="0.1524" layer="91"/>
-<pinref part="X1" gate="G$1" pin="6"/>
 <wire x1="-40.64" y1="-60.96" x2="-38.1" y2="-60.96" width="0.1524" layer="91"/>
-<pinref part="X2" gate="G$1" pin="3"/>
 <wire x1="-22.86" y1="-53.34" x2="-25.4" y2="-53.34" width="0.1524" layer="91"/>
 <wire x1="-25.4" y1="-53.34" x2="-25.4" y2="-60.96" width="0.1524" layer="91"/>
-<pinref part="X2" gate="G$1" pin="6"/>
 <wire x1="-25.4" y1="-60.96" x2="-22.86" y2="-60.96" width="0.1524" layer="91"/>
 <wire x1="-38.1" y1="-60.96" x2="-25.4" y2="-60.96" width="0.1524" layer="91"/>
@@
 <junction x="-40.64" y="-60.96"/>
 <junction x="-38.1" y="-60.96"/>
+<pinref part="X3" gate="G$1" pin="3"/>
+<pinref part="X3" gate="G$1" pin="6"/>
+<pinref part="X1" gate="G$1" pin="3"/>
+<pinref part="X1" gate="G$1" pin="6"/>
 </segment>
 <segment>
@@
 </segment>
 <segment>
-<pinref part="X1" gate="G$1" pin="4"/>
-<pinref part="X1" gate="G$1" pin="5"/>
 <wire x1="-38.1" y1="-55.88" x2="-38.1" y2="-58.42" width="0.1524" layer="91"/>
-<pinref part="X2" gate="G$1" pin="4"/>
-<pinref part="X2" gate="G$1" pin="5"/>
 <wire x1="-22.86" y1="-55.88" x2="-22.86" y2="-58.42" width="0.1524" layer="91"/>
 <wire x1="-38.1" y1="-58.42" x2="-27.94" y2="-58.42" width="0.1524" layer="91"/>
@@
 <wire x1="-27.94" y1="-58.42" x2="-22.86" y2="-58.42" width="0.1524" layer="91"/>
 <junction x="-27.94" y="-58.42"/>
+<pinref part="X3" gate="G$1" pin="4"/>
+<pinref part="X3" gate="G$1" pin="5"/>
+<pinref part="X1" gate="G$1" pin="4"/>
+<pinref part="X1" gate="G$1" pin="5"/>
 </segment>
 </net>
@@
 <pinref part="R11" gate="G$1" pin="2"/>
 <wire x1="-53.34" y1="-53.34" x2="-48.26" y2="-53.34" width="0.1524" layer="91"/>
-<pinref part="X1" gate="G$1" pin="1"/>
 <wire x1="-38.1" y1="-48.26" x2="-53.34" y2="-48.26" width="0.1524" layer="91"/>
 <wire x1="-53.34" y1="-48.26" x2="-53.34" y2="-53.34" width="0.1524" layer="91"/>
 <junction x="-53.34" y="-53.34"/>
-<pinref part="X2" gate="G$1" pin="1"/>
 <wire x1="-22.86" y1="-48.26" x2="-38.1" y2="-48.26" width="0.1524" layer="91"/>
 <junction x="-38.1" y="-48.26"/>
+<pinref part="X3" gate="G$1" pin="1"/>
+<pinref part="X1" gate="G$1" pin="1"/>
 </segment>
 </net>
@@
 <junction x="-48.26" y="-63.5"/>
 <wire x1="-45.72" y1="-63.5" x2="-45.72" y2="-50.8" width="0.1524" layer="91"/>
-<pinref part="X1" gate="G$1" pin="2"/>
 <wire x1="-45.72" y1="-50.8" x2="-38.1" y2="-50.8" width="0.1524" layer="91"/>
-<pinref part="X2" gate="G$1" pin="2"/>
 <wire x1="-38.1" y1="-50.8" x2="-22.86" y2="-50.8" width="0.1524" layer="91"/>
 <junction x="-38.1" y="-50.8"/>
-</segment>
-</net>
+<pinref part="X3" gate="G$1" pin="2"/>
+<pinref part="X1" gate="G$1" pin="2"/>
+</segment>
+</net>

Commit message: add values
Parts:
- C1, C11, C14, C15, C16, C17, C18, C19, C20, C21, C22, C23, C24, C25, C26, C3, C4, C5, C7, C8, C9: value (none) -> 0.1uF
- C10: value (none) -> 10nF
- C12, C2, C6: value (none) -> 10uF
- R1, R10, R5, R6, R7: value (none) -> 10K
- R11: value (none) -> 120
- R12, R13: value (none) -> 1K
- R2, R3, R4: value (none) -> DNP
- R8, R9: value (none) -> 51K

Commit message: add value and gerber
Parts:
- D1, D19, D2, D3, D4, D5, D6: value (none) -> 5819
- U3: value MAX3485CSA -> SP485
Changed lines of the file:
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@@
 <part name="R4" library="resistor" library_urn="urn:adsk.eagle:library:348" deviceset="R-US_" device="R0805" package3d_urn="urn:adsk.eagle:package:26059/1" value="DNP"/>
 <part name="J5" library="SparkFun-Connectors" deviceset="CONN_01" device=""/>
-<part name="D1" library="adafruit" library_urn="urn:adsk.eagle:library:420" deviceset="DIODE" device="SOD-123"/>
+<part name="D1" library="adafruit" library_urn="urn:adsk.eagle:library:420" deviceset="DIODE" device="SOD-123" value="5819"/>
 <part name="R5" library="resistor" library_urn="urn:adsk.eagle:library:348" deviceset="R-US_" device="R0805" package3d_urn="urn:adsk.eagle:package:26059/1" value="10K"/>
 <part name="+3V2" library="supply1" library_urn="urn:adsk.eagle:library:371" deviceset="+3V3" device=""/>
-<part name="D2" library="adafruit" library_urn="urn:adsk.eagle:library:420" deviceset="DIODE" device="SOD-123"/>
-<part name="D3" library="adafruit" library_urn="urn:adsk.eagle:library:420" deviceset="DIODE" device="SOD-123"/>
-<part name="D4" library="adafruit" library_urn="urn:adsk.eagle:library:420" deviceset="DIODE" device="SOD-123"/>
+<part name="D2" library="adafruit" library_urn="urn:adsk.eagle:library:420" deviceset="DIODE" device="SOD-123" value="5819"/>
+<part name="D3" library="adafruit" library_urn="urn:adsk.eagle:library:420" deviceset="DIODE" device="SOD-123" value="5819"/>
+<part name="D4" library="adafruit" library_urn="urn:adsk.eagle:library:420" deviceset="DIODE" device="SOD-123" value="5819"/>
 <part name="R6" library="resistor" library_urn="urn:adsk.eagle:library:348" deviceset="R-US_" device="R0805" package3d_urn="urn:adsk.eagle:package:26059/1" value="10K"/>
 <part name="+3V3" library="supply1" library_urn="urn:adsk.eagle:library:371" deviceset="+3V3" device=""/>
 <part name="R7" library="resistor" library_urn="urn:adsk.eagle:library:348" deviceset="R-US_" device="R0805" package3d_urn="urn:adsk.eagle:package:26059/1" value="10K"/>
 <part name="+3V6" library="supply1" library_urn="urn:adsk.eagle:library:371" deviceset="+3V3" device=""/>
-<part name="D5" library="adafruit" library_urn="urn:adsk.eagle:library:420" deviceset="DIODE" device="SOD-123"/>
-<part name="D6" library="adafruit" library_urn="urn:adsk.eagle:library:420" deviceset="DIODE" device="SOD-123"/>
-<part name="U3" library="SparkFun-IC-Comms" deviceset="RS485" device="SOIC" value=" MAX3485CSA"/>
+<part name="D5" library="adafruit" library_urn="urn:adsk.eagle:library:420" deviceset="DIODE" device="SOD-123" value="5819"/>
+<part name="D6" library="adafruit" library_urn="urn:adsk.eagle:library:420" deviceset="DIODE" device="SOD-123" value="5819"/>
+<part name="U3" library="SparkFun-IC-Comms" deviceset="RS485" device="SOIC" value="SP485"/>
 <part name="D7" library="SparkFun-LED" library_urn="urn:adsk.eagle:library:529" deviceset="WS2812B" device="" package3d_urn="urn:adsk.eagle:package:39369/1" value="WS2812B"/>
 <part name="D8" library="SparkFun-LED" library_urn="urn:adsk.eagle:library:529" deviceset="WS2812B" device="" package3d_urn="urn:adsk.eagle:package:39369/1" value="WS2812B"/>
@@
 <part name="IC2" library="lmrdcdc-0.1" deviceset="LMR16006" device="X" value="MP2359"/>
 <part name="L1" library="SparkFun-Coils" deviceset="INDUCTOR" device="-IFSC1515AHER2R2M01" value="4.7uH"/>
-<part name="D19" library="adafruit" library_urn="urn:adsk.eagle:library:420" deviceset="DIODE" device="SOD-123"/>
+<part name="D19" library="adafruit" library_urn="urn:adsk.eagle:library:420" deviceset="DIODE" device="SOD-123" value="5819"/>
 <part name="C10" library="resistor" library_urn="urn:adsk.eagle:library:348" deviceset="C-EU" device="C0805K" package3d_urn="urn:adsk.eagle:package:26201/1" value="10nF"/>
 <part name="R8" library="resistor" library_urn="urn:adsk.eagle:library:348" deviceset="R-US_" device="R0805" package3d_urn="urn:adsk.eagle:package:26059/1" value="51K"/>

Commit message: add note
Other:
- note added: "Todo: Add pull up resistor on RX due to HiZ of SP485"
Changed lines of the file:
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@@
 <?xml version="1.0" encoding="utf-8"?>
 <!DOCTYPE eagle SYSTEM "eagle.dtd">
-<eagle version="8.3.2">
+<eagle version="8.5.1">
 <drawing>
 <settings>
@@
 <sheet>
 <plain>
+<text x="129.54" y="-55.88" size="6.4516" layer="91">Todo:
+Add pull up resistor on RX due to HiZ of SP485</text>
 </plain>
 <instances>
@@
 </drawing>
 <compatibility>
+<note version="6.3" minversion="6.2.2" severity="warning">
+Since Version 6.2.2 text objects can contain more than one line,
+which will not be processed correctly with this version.
+</note>
 <note version="8.2" severity="warning">
 Since Version 8.2, EAGLE supports online libraries. The ids

Commit message: add resistor
Parts:
- added R14: 10K, resistor:R-US_R0805
Connections:
- net +5V: now also R14.2
- net RX: now also R14.1
Changed lines of the file:
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@@
 <?xml version="1.0" encoding="utf-8"?>
 <!DOCTYPE eagle SYSTEM "eagle.dtd">
-<eagle version="8.5.1">
+<eagle version="8.7.0">
 <drawing>
 <settings>
@@
 <part name="X3" library="myownParts" deviceset="RJ45-8P8C" device="" technology="-8L-B"/>
 <part name="X1" library="myownParts" deviceset="RJ45-8P8C" device="" technology="-8L-B"/>
+<part name="R14" library="resistor" library_urn="urn:adsk.eagle:library:348" deviceset="R-US_" device="R0805" package3d_urn="urn:adsk.eagle:package:26059/1" value="10K"/>
+<part name="P+10" library="supply1" library_urn="urn:adsk.eagle:library:371" deviceset="+5V" device=""/>
 </parts>
 <sheets>
@@
 <instance part="C24" gate="G$1" x="-66.04" y="-5.08"/>
 <instance part="C25" gate="G$1" x="-66.04" y="-25.4"/>
-<instance part="P+20" gate="1" x="-55.88" y="-50.8"/>
+<instance part="P+20" gate="1" x="-55.88" y="-50.8" smashed="yes">
+<attribute name="VALUE" x="-58.42" y="-50.8" size="1.778" layer="96"/>
+</instance>
 <instance part="GND27" gate="1" x="-55.88" y="-63.5"/>
 <instance part="R11" gate="G$1" x="-48.26" y="-58.42" rot="R90"/>
@@
 <instance part="X3" gate="G$1" x="-35.56" y="-55.88"/>
 <instance part="X1" gate="G$1" x="-20.32" y="-55.88"/>
+<instance part="R14" gate="G$1" x="-88.9" y="-45.72"/>
+<instance part="P+10" gate="1" x="-83.82" y="-43.18" smashed="yes">
+<attribute name="VALUE" x="-83.82" y="-43.18" size="1.778" layer="96"/>
+</instance>
 </instances>
 <busses>
@@
 <wire x1="-93.98" y1="-53.34" x2="-99.06" y2="-53.34" width="0.1524" layer="91"/>
 <label x="-99.06" y="-53.34" size="1.778" layer="95"/>
+<pinref part="R14" gate="G$1" pin="1"/>
+<wire x1="-93.98" y1="-53.34" x2="-93.98" y2="-45.72" width="0.1524" layer="91"/>
+<junction x="-93.98" y="-53.34"/>
 </segment>
 </net>
@@
 <junction x="-106.68" y="78.74"/>
 </segment>
-</net>
+<segment>
+<pinref part="R14" gate="G$1" pin="2"/>
+<pinref part="P+10" gate="1" pin="+5V"/>
+</segment>
+</net>

Commit message: 48V upgrade
Parts:
- removed C11: 0.1uF, resistor:C-EUC0805K
- removed D19: 5819, adafruit:DIODESOD-123
- added C27, C28, C29, C30, C31, C32, C33, C34, C35: 1uF 100V, SparkFun-Capacitors:10UF-1206-6.3V-20%
- added C36: 150pF, resistor:C-EUC0805K
- added C38: 10uF, resistor:C-EUC0805K
- added D20: B280-13-F, diode:DIODE-DO214AA
- added R15: 17.4K, resistor:R-US_R0805
- added R16: 200K, resistor:R-US_R0805
- added R17: 158K, resistor:R-US_R0805
- C10: value 10nF -> 0.1uF
- C13: value 10uF -> 1uF 100V; LCSC (none) -> C91151
- IC2: value MP2359 -> MP2562; device lmrdcdc-0.1:LMR16006X -> misc:MP2562; LCSC (none) -> C93647
- L1: value 4.7uH -> 15uH; device SparkFun-Coils:INDUCTOR-IFSC1515AHER2R2M01 -> misc:SLF12575T
- R10: value 10K -> 40.2k
- R8: value 51K -> 100K
- R9: value 51K -> 210K
Connections:
- net N$21 renamed FB
- removed net N$18: C10.2, D19.C, IC2.SW, L1.1
- removed net N$19: C10.1, IC2.CB
- removed net N$23: IC2.!SHDN, R8.1
- new net BST: C10.1, IC2.BST
- new net COMP: C36.1, IC2.COMP
- new net EN: IC2.EN, R15.2, R8.1
- new net FREQ: IC2.FREQ, R16.2
- new net N$25: C36.2, R17.2
- new net SW: C10.2, D20.C, IC2.SW, L1.1
- net +24V: now also C27.1, C28.1, C29.1, C30.1, C31.1, C32.1, C33.1, C34.1, C35.1
- net +5V: now also C38.1; no longer C11.1
- net GND: now also C27.2, C28.2, C29.2, C30.2, C31.2, C32.2, C33.2, C34.2, C35.2, C38.2, D20.A, R15.1, R16.1, R17.1; no longer C11.2, D19.A
Other:
- note removed: "Todo: Add pull up resistor on RX due to HiZ of SP485"
- moved on the sheet: C10, C12, C13, R10, R8, R9
