File: Eagle Files/rs485board/rs485board.sch (EAGLE design)
At the start: 95 parts, among them IC1 XC6206P332MR, IC2 MP2562, J1 AVR_SPI_PROG_3X2PTH, J2 RA 6Pin SMD, Q1 CJ3404, Q2 CJ3404, Q3 CJ3404, U1 ATMEGA328P_TQFP, U2 LIS3DH, U3 SP485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

Commit message: add lcsc part number
Parts:
- C1, C10, C14, C15, C16, C17, C18, C19, C20, C21, C22, C23, C24, C25, C26, C3, C4, C5, C7, C8, C9: LCSC (none) -> C29926
- C12, C2, C38, C6: LCSC (none) -> C92341
- C36: LCSC (none) -> C152846
- D1, D2, D3, D4, D5, D6: LCSC (none) -> C64885
- D10, D11, D12, D13, D14, D15, D16, D17, D18, D7, D8, D9: LCSC (none) -> C114585
- IC1: LCSC (none) -> C5446
- L1: LCSC (none) -> C136211
- R1, R14, R5, R6, R7: LCSC (none) -> C17414
- R10: LCSC (none) -> C104303
- R12, R13: LCSC (none) -> C115316
- R15: LCSC (none) -> C144583
- R16: LCSC (none) -> C17539
- R17: LCSC (none) -> C104013
- R8: LCSC (none) -> C96346
- R9: LCSC (none) -> C170839
- U1: LCSC (none) -> C14877
- U2: LCSC (none) -> C15134
- U3: LCSC (none) -> C6855
- X1, X3: LCSC (none) -> C86586
- Y1: LCSC (none) -> C91584
